File: schema/jrr5/jrr5.kicad_pcb (KiCad board)
At the start: 2 copper layers, 110 x 56 mm, 39 parts, among them J11 Wafer,1x2,m, J13 Wafer,1x2,m, J18 Wafer,1x3,m, J19 Wafer,1x2,m, J2 Raspberry_Pi_2_3_GPIO, J21 Wafer,1x2,m, J24 Wafer,1x2,m, J26 Wafer,1x3,m, J28 Wafer,1x2,m, J3 USB-C,6Pin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

Commit message: dev
Parts:
- TP4: value DAC-IN -> Dac-In
- TP6: value Audio-in -> AUDIO-IN
- moved SW1 15.0 mm to (-25.8, 17.8)
- moved SW2 15.0 mm to (-25.8, 33.8)
- moved J24 10.6 mm to (-9.77, 27.4)
- moved JP2 10.1 mm to (-14.9, 35.7)
- moved TP2 7.16 mm to (-27.5, 12.9)
- moved TP8 6.15 mm to (-9.18, 46.4)
- moved TP4 5.15 mm to (-3.86, 46.2)
- moved TP5 4.24 mm to (-26.7, 51.1)
- moved J13 2.83 mm to (-17.6, 43.8)
- moved TP7 1.66 mm to (-2.64, 26.9), turned to -90 degrees
Routing:
- net Net-(J2-GPIO20/MOSI1): track 99.2 -> 114.2 mm
- net Net-(J2-GPIO19/MISO1): track 69.5 -> 84.5 mm
- net +5V-RPI: track 94.9 -> 90.2 mm
- net +5V-IN: track 47.5 -> 43.5 mm
- net RCA-IN: track 11.7 -> 8.35 mm
- net audio-in: track 15.2 -> 13.1 mm
- net DAC-IN: track 22.6 -> 20.6 mm
Other:
- board text added: "DAC-IN"
- board text added: "Rca-In"
- board text removed: "RCA-IN"
