File: schema/jrr5/jrr5.kicad_sch (KiCad schematic)
At the start: 64 parts, among them J1 3.5inc TFT display, J101 Wafer,1x2,m, J102 Wafer,1x2,fm, J103 Wafer,1x2,fm, J104 Wafer,1x2,m, J105 Wafer,1x2,fm, J106 Wafer,1x2,m, J107 Wafer,1x2,fm, J108 Wafer,1x2,fm, J109 Wafer,1x3,fm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

Commit message: JRR-14: R1/R2 100k->10k
Parts:
- R1, R2: value 100k -> 10k
